File: pico-HABakuk.kicad_sch (KiCad schematic)
At the start: 78 parts, among them J1 USB_B_Micro, J2 Ant+, J3 GPS Ant, J4 Ant-, J5 Solar, J6 Debug, J7 Super_Cap, Q1 BSS84, SW1 USB BOOT, SW2 RESET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

Commit message: board finetuning, GPIO pins added
Parts:
- added H1, H2: MountingHole, MountingHole:MountingHole_2.1mm, symbol Mechanical:MountingHole
- added TP17: 10, TestPoint:TestPoint_THTPad_D1.0mm_Drill0.5mm, symbol Connector:TestPoint
- added TP18: 11, TestPoint:TestPoint_THTPad_D1.0mm_Drill0.5mm, symbol Connector:TestPoint
- added TP19: 12, TestPoint:TestPoint_THTPad_D1.0mm_Drill0.5mm, symbol Connector:TestPoint
- added TP20: 13, TestPoint:TestPoint_THTPad_D1.0mm_Drill0.5mm, symbol Connector:TestPoint
- added TP21: gnd, TestPoint:TestPoint_THTPad_D1.0mm_Drill0.5mm, symbol Connector:TestPoint
- added TP22: +, TestPoint:TestPoint_THTPad_D1.0mm_Drill0.5mm, symbol Connector:TestPoint
- added TP23: AD0, TestPoint:TestPoint_THTPad_D1.0mm_Drill0.5mm, symbol Connector:TestPoint
Connections:
- net +3V3: now also TP22.1
- net GND: now also TP21.1
- net GPIO10: now also TP17.1
- net GPIO11: now also TP18.1
- net GPIO12: now also TP19.1
- net GPIO13: now also TP20.1
- net GPIO26_ADC0: now also TP23.1

Commit message: Final board tuning and DRC debuging
Parts:
- added C26, C27: 10u, Capacitor_SMD:C_0805_2012Metric, symbol Device:C
- added R14: 2k2, Resistor_SMD:R_0603_1608Metric, symbol Device:R
- TP10: value USB_D+ -> D+
- TP11: value USB_D- -> D-
- TP12: value GND -> gnd
- TP13: value USB_BOOT -> boot
- TP14: value Reset -> rst
- TP15: value SWCLK -> swclk
- TP16: value SWD -> swd
- TP9: value +3V3 -> +
Connections:
- net +3V3: now also C26.1, C27.1
- net GND: now also C26.2, C27.2
- net RUN: now also R14.1; no longer U7.2 (~{RESET})
- new net: R14.2, U7.2 (~{RESET})

Commit message: Minor silkscreen edits
Parts:
- JP1: value Solar_voltage -> sol adc2
- JP2: value GPS+Glonass -> GPS opt
Changed lines of the file:
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@@
 			)
 		)
-		(property "Value" "GPS+Glonass"
+		(property "Value" "GPS opt"
 			(at 316.23 129.54 0)
 			(effects
@@
 			)
 		)
-		(property "Value" "Solar_voltage"
+		(property "Value" "sol adc2"
 			(at 43.18 31.7499 90)
 			(effects
